File: ProjetVenus/ProjetVenus.kicad_pcb (KiCad board)
At the start: 2 copper layers, 60 x 37.5 mm, 44 parts, among them J1 Conn_01x02_Pin, J2 Conn_01x04_Pin, J4 Conn_01x02_Pin, J5 Conn_01x05_Pin, Q1 Q_NMOS_GSD, U1 ATtiny412-SS, U2 ADP2108AUJZ-3.0-R7, U3 MS5607-02BA

Commit message: V1.1
Parts:
- added H1: MountingHole, MountingHole:MountingHole_3.2mm_M3_Pad_Via, F.Cu at (245.8, 90.0)
- added H2: MountingHole, MountingHole:MountingHole_3.2mm_M3_Pad_Via, F.Cu at (190.9, 90.0)
- added H3: MountingHole, MountingHole:MountingHole_3.2mm_M3_Pad_Via, F.Cu at (190.9, 122.7)
- added H4: MountingHole, MountingHole:MountingHole_3.2mm_M3_Pad_Via, F.Cu at (245.8, 122.7)
- moved TP2 2.65 mm to (240.1, 94.1)
Routing:
- net +3V0: track 164.0 -> 140.7 mm, vias 17 -> 0
- net GND: track 222.7 -> 207.7 mm
Other:
- board size 60 x 37.5 mm -> 66.3 x 44.1 mm

Commit message: V1.2
Parts:
- H1, H2, H3, H4: value MountingHole -> MountingHole_Pad; footprint MountingHole:MountingHole_3.2mm_M3_Pad_Via -> MountingHole:MountingHole_3.2mm_M3_DIN965_Pad
- moved H2 55.6 mm to (246.5, 89.5)
- moved H1 55.4 mm to (190.4, 89.8)
- moved H4 55.1 mm to (190.8, 123.2)
- moved H3 54.9 mm to (245.8, 123.0)
- moved TP4 24.5 mm to (232.5, 104.8)
- moved R17 18.0 mm to (211.0, 98.1), turned to -90 degrees
- moved R16 16.2 mm to (221.0, 98.8), turned to 90 degrees
- moved J1 12.4 mm to (227.0, 90.8)
- moved R3 10.6 mm to (229.8, 122.5), turned to 90 degrees
- moved R2 9.45 mm to (231.5, 119.0), turned to 90 degrees
- moved C8 9.25 mm to (239.2, 119.8), turned to 180 degrees
- moved J4 7.75 mm to (221.0, 90.8)
- moved C7 7.64 mm to (239.3, 122.8), turned to 0 degrees
- moved TP1 5.88 mm to (232.4, 94.8)
- moved D3 0.93 mm to (200.6, 93.3)
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Connections:
- H1 pad 1: (no net) -> unconnected-(H1-Pad1)
- H2 pad 1: GND -> unconnected-(H2-Pad1)
- H3 pad 1: (no net) -> unconnected-(H3-Pad1)
- H4 pad 1: (no net) -> unconnected-(H4-Pad1)
Routing:
- net GND: track 207.7 -> 56.5 mm, vias 30 -> 34
- net +3V0: track 140.7 -> 17.3 mm, vias 0 -> 4
- net /SDA: track 66.4 -> 131.2 mm
- net +BATT: track 52.4 -> 0.00 mm
- net /EMATCH_DET: track 16.2 -> 34.8 mm
- net Net-(J4-Pin_1): track 44.9 -> 53.5 mm
- net /SCL: track 49.1 -> 43.1 mm
- net /UPDI: track 21.0 -> 19.4 mm
- net /EMATCH: track 27.6 -> 26.4 mm
- added copper zone on F.Cu, net +3V0
- added copper zone on F.Cu, net +BATT
